File: pcb/MGC.kicad_pcb (KiCad board)
At the start: 2 copper layers, 92.7 x 62.2 mm, 121 parts, among them J1 USB_C_Receptacle, J10 Conn_01x04_Pin, J11 103R012BB100, J12 103R012BB100, J13 103R012BB100, J14 Conn_02x10_Odd_Even, J15 Conn_02x10_Odd_Even, J16 Conn_01x03, J17 Conn_01x01_Pin, J18 Conn_01x02_Pin, J19 Conn_01x02_Pin, J2 Conn_01x02_Pin, J20 Conn_01x02_Pin, J3 103R012BB100, J4 Conn_02x03_Odd_Even, J5 Conn_02x05_Odd_Even, J6 Conn_01x04, J7 103R012BB100, J8 Conn_01x01_Pin, J9 Conn_01x01_Pin, Q10 AO3416, Q11 AO3416, Q12 AO3416, Q13 AO3416, Q9 AO3416, SW0 SW_SPST, SW1 SW_SPST, SW2 SW_SPST, SW3 SW_SPST, SW5 SW_SPST, SW6 SW_DIP_x02, U1 FT230XS, U2 TS3USB30EDGSR, U3 74AHC1G14, U4 TPS2116DRL, U5 LM1117DT-3.3, U6 TBD62783A, U7 MB85RC04V

Commit message: Add missing dimensions
Other:
- board text added: "V_POT"
- board text removed: "VPOT"
Changed lines of the file:
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@@
 		)
 	)
-	(gr_text "VPOT"
+	(gr_text "V_POT"
 		(at 140.97 124.841 0)
 		(layer "F.SilkS")
@@
 	(dimension
 		(type orthogonal)
+		(layer "Dwgs.User")
+		(pts
+			(xy 170.434 89.408) (xy 101.6 89.408)
+		)
+		(height 51.562)
+		(orientation 0)
+		(format
+			(prefix "")
+			(suffix "")
+			(units 3)
+			(units_format 0)
+			(precision 2)
+			(suppress_zeroes yes)
+		)
+		(style
+			(thickness 0.15)
+			(arrow_length 1.27)
+			(text_position_mode 0)
+			(arrow_direction outward)
+			(extension_height 0.58642)
+			(extension_offset 0.5)
+			(keep_text_aligned yes)
+		)
+		(gr_text "68.83"
+			(at 136.017 139.82 0)
+			(layer "Dwgs.User")
+			(effects
+				(font
+					(size 1 1)
+					(thickness 0.15)
+				)
+			)
+		)
+	)
+	(dimension
+		(type orthogonal)
 		(layer "User.1")
 		(pts
@@
 			(xy 170.1754 124.6454) (xy 101.6 124.6454)
 		)
-		(height 36.6446)
+		(height 39.1846)
 		(orientation 0)
 		(format
@@
 		)
 		(gr_text "68.58"
-			(at 135.8877 160.14 0)
+			(at 135.8877 162.68 0)
 			(layer "User.1")
 			(effects
@@
 			(xy 144.325 70.485) (xy 101.6 70.485)
 		)
-		(height 75.565)
+		(height 78.105)
 		(orientation 0)
 		(format
@@
 		)
 		(gr_text "42.73"
-			(at 122.9625 144.9 0)
+			(at 122.9625 147.44 0)
 			(layer "User.1")
 			(effects
@@
 			(xy 153.85 70.485) (xy 101.6 70.485)
 		)
-		(height 85.725)
+		(height 88.265)
 		(orientation 0)
 		(format
@@
 		)
 		(gr_text "52.25"
-			(at 127.725 155.06 0)
+			(at 127.725 157.6 0)
 			(layer "User.1")
 			(effects
@@
 		(layer "User.1")
 		(pts
+			(xy 140.97 122.428) (xy 101.6 122.428)
+		)
+		(height 23.622)
+		(orientation 0)
+		(format
+			(prefix "")
+			(suffix "")
+			(units 3)
+			(units_format 0)
+			(precision 2)
+			(suppress_zeroes yes)
+		)
+		(style
+			(thickness 0.15)
+			(arrow_length 1.27)
+			(text_position_mode 0)
+			(arrow_direction outward)
+			(extension_height 0.58642)
+			(extension_offset 0.5)
+			(keep_text_aligned yes)
+		)
+		(gr_text "39.37"
+			(at 121.285 144.9 0)
+			(layer "User.1")
+			(effects
+				(font
+					(size 1 1)
+					(thickness 0.15)
+				)
+			)
+		)
+	)
+	(dimension
+		(type orthogonal)
+		(layer "User.1")
+		(pts
 			(xy 106.68 96.52) (xy 101.6 96.52)
 		)
@@
 		(layer "User.1")
 		(pts
+			(xy 179.324 67.31) (xy 101.6 67.31)
+		)
+		(height -12.7)
+		(orientation 0)
+		(format
+			(prefix "")
+			(suffix "")
+			(units 3)
+			(units_format 0)
+			(precision 2)
+			(suppress_zeroes yes)
+		)
+		(style
+			(thickness 0.15)
+			(arrow_length 1.27)
+			(text_position_mode 0)
+			(arrow_direction outward)
+			(extension_height 0.58642)
+			(extension_offset 0.5)
+			(keep_text_aligned yes)
+		)
+		(gr_text "77.72"
+			(at 140.462 53.46 0)
+			(layer "User.1")
+			(effects
+				(font
+					(size 1 1)
+					(thickness 0.15)
+				)
+			)
+		)
+	)
+	(dimension
+		(type orthogonal)
+		(layer "User.1")
+		(pts
 			(xy 180.086 80.3616) (xy 101.6 80.3616)
 		)
-		(height -25.7516)
+		(height -28.2916)
 		(orientation 0)
 		(format
@@
 		)
 		(gr_text "78.49"
-			(at 140.843 53.46 0)
+			(at 140.843 50.92 0)
 			(layer "User.1")
 			(effects
@@
 			(xy 149.86 110.105) (xy 101.6 110.105)
 		)
-		(height 41.025)
+		(height 43.565)
 		(orientation 0)
 		(format
@@
 		)
 		(gr_text "48.26"
-			(at 125.73 149.98 0)
+			(at 125.73 152.52 0)
 			(layer "User.1")
 			(effects
@@
 			(xy 166.37 70.485) (xy 101.6 70.485)
 		)
-		(height 88.265)
+		(height 90.805)
 		(orientation 0)
 		(format
@@
 		)
 		(gr_text "64.77"
-			(at 133.985 157.6 0)
+			(at 133.985 160.14 0)
 			(layer "User.1")
 			(effects
@@
 			(xy 149.272335 119.653239) (xy 101.6 119.653239)
 		)
-		(height 28.936761)
+		(height 31.476761)
 		(orientation 0)
 		(format
@@
 		)
 		(gr_text "47.67"
-			(at 126.492 147.447 0)
+			(at 126.492 149.987 0)
 			(layer "User.1")
 			(effects
@@
 			(xy 181.75 90.17) (xy 101.6 90.17)
 		)
-		(height -38.1)
+		(height -40.64)
 		(orientation 0)
 		(format
@@
 		)
 		(gr_text "80.15"
-			(at 141.675 50.92 0)
+			(at 141.675 48.38 0)
 			(layer "User.1")
 			(effects
@@
 			(xy 189.91 87.63) (xy 101.6 87.63)
 		)
-		(height -38.1)
+		(height -40.64)
 		(orientation 0)
 		(format
@@
 		)
 		(gr_text "88.31"
-			(at 145.755 48.38 0)
+			(at 145.755 45.84 0)
 			(layer "User.1")
 			(effects
@@
 		(layer "User.1")
 		(pts
+			(xy 140.97 122.428) (xy 140.97 63.5)
+		)
+		(height 76.2)
+		(orientation 1)
+		(format
+			(prefix "")
+			(suffix "")
+			(units 3)
+			(units_format 0)
+			(precision 2)
+			(suppress_zeroes yes)
+		)
+		(style
+			(thickness 0.15)
+			(arrow_length 1.27)
+			(text_position_mode 0)
+			(arrow_direction outward)
+			(extension_height 0.58642)
+			(extension_offset 0.5)
+			(keep_text_aligned yes)
+		)
+		(gr_text "58.93"
+			(at 216.02 92.964 90)
+			(layer "User.1")
+			(effects
+				(font
+					(size 1 1)
+					(thickness 0.15)
+				)
+			)
+		)
+	)
+	(dimension
+		(type orthogonal)
+		(layer "User.1")
+		(pts
 			(xy 157.48 94.88) (xy 101.6 94.88)
 		)
@@
 			(xy 150.495 102.342) (xy 101.6 102.342)
 		)
-		(height 51.328)
+		(height 53.868)
 		(orientation 0)
 		(format
@@
 		)
 		(gr_text "48.9"
-			(at 126.0475 152.52 0)
-			(layer "User.1")
-			(effects
+			(at 126.0475 155.06 0)
+			(layer "User.1")
+			(effects
